File: schematics/debug.kicad_sch (KiCad schematic)
At the start: 5 parts, among them J2 PinHeader_1x2_P2.54mm_Drill1.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, J4 PinHeader_2x7_P2mm_Drill1mm_S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, U14 TPD4E05U06QDQARQ1, U2 TXS0102DCU

Commit message: Voltage converter added
Parts:
- removed U2: TXS0102DCU, Package_SO:VSSOP-8_2.3x2mm_P0.5mm, symbol Logic_LevelTranslator:TXS0102DCU
- added U12: TXS0102DCU, Package_SO:VSSOP-8_2.3x2mm_P0.5mm, symbol Logic_LevelTranslator:TXS0102DCU
- renumbered C52 to C43, J2 to J4, J4 to J5, U14 to U13
Connections:
- net CONN_GND is gone; now on net ~{PS_SRST_C2M}: J5.14
- net GND: now also U12.2 (GND)
- net MIO36: now also U12.5 (A1)
- net MIO37: now also U12.4 (A2)
- net PS_1V8: now also U12.3 (VCCA), U12.6 (OE)
- net PS_3V3: now also U12.7 (VCCB)
- net ~{PS_SRST_C2M}: no longer J5.13
- net at J4.2: now also U12.1 (B2)
- net at J4.1: now also U12.8 (B1)
Other:
- moved on the sheet: J5
