File: schematics/k26_som.kicad_sch (KiCad schematic)
At the start: 41 parts, among them M1 XILINX-KRIA-K26

Commit message: Voltage converter added
Parts:
- J_SOM240_3: renamed from J_SOM240_1; Pitch (none) -> 0.635 mm
- J_SOM240_4: renamed from J_SOM240_2; DNP DNP -> (none); Pitch (none) -> 0.635 mm; now in the parts list
- M1: Manufacturer Xilinx -> AMD-Xilinx
- R51: renamed from R72; DNP DNP -> (none); now in the parts list
- TP13: renamed from TP28; now left out of the parts list
- TP14: renamed from TP29; now left out of the parts list
- TP15: renamed from TP30; now left out of the parts list
- TP16: renamed from TP31; now left out of the parts list
- TP17: renamed from TP32; now left out of the parts list
- TP18: renamed from TP33; now left out of the parts list
- TP19: renamed from TP34; now left out of the parts list
- TP20: renamed from TP35; now left out of the parts list
- renumbered C68 to C52, C69 to C53, C70 to C54, C71 to C55, C72 to C56, C73 to C57, C74 to C58, C75 to C59, C76 to C60, C77 to C61, C78 to C62, C79 to C63, C80 to C64, C81 to C65, C82 to C66, R69 to R48, R70 to R49, R71 to R50, R73 to R52, R74 to R53
Connections:
- net GND: now also S2.2; no longer S2.3
- net MIO12_FWUEN_C2M_L: now also S2.3; no longer S2.2
- net HDA00_C renamed HDA00_CC
Other:
- note added: "SOM K26 connectors"
- note removed: "SOM K26 B2B connectors"
- moved on the sheet: C52, C53, C54, C55, C56, C57, C58, C59, C60, C61, C62, C63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
