File: schematics/mezzanine_connectors.kicad_sch (KiCad schematic)
At the start: 3 parts

Commit message: Voltage converter added
Parts:
- J_SOM240_1: renamed from J_SOM240_3; Pitch (none) -> 0.635 mm
- J_SOM240_2: renamed from J_SOM240_4; DNP DNP -> (none); Pitch (none) -> 0.635 mm; now in the parts list
- renumbered R96 to R36
Connections:
- net MIO76: now reaches J_SOM240_1.D44
- net MIO77: now reaches J_SOM240_1.D45
- net HDA00_C renamed HDA00_CC
- net HDA01 renamed MEZZ_RST_N
- net HDA02: no longer names the net of J_SOM240_1.D18
- net MIO40: no longer names the net of J_SOM240_1.B34
- net MIO42: no longer names the net of J_SOM240_1.A35
- net ~{PS_SRST_C2M}: no longer names the net of J_SOM240_1.C16
