File: schematics/reset.kicad_sch (KiCad schematic)
At the start: 33 parts, among them Q5 DTC014T_SOT-416, Q6 DTC014T_SOT-416, U17 TPS3840PH30DBVR, U18 TPS3840PH30DBVR, U19 74AVC4T245_UQFN, U20 SN74LVC1G125_SOT, U21 74LCX07_QFN

Commit message: Voltage converter added
Parts:
- removed R68, R95: R_10k_0402, kria-k26-devboard-footprints:R_0402_1005Metric, symbol kria-k26-devboard:R_10k_0402
- added C126: C_220n_0402, kria-k26-devboard-footprints:C_0402_1005Metric, symbol kria-k26-devboard:C_47n_0402
- added C127: C_100n_0402, kria-k26-devboard-footprints:C_0402_1005Metric, symbol kria-k26-devboard:C_100n_0402
- added R46, R47: R_10k_0402, kria-k26-devboard-footprints:R_0402_1005Metric, symbol kria-k26-devboard:R_10k_0402
- added TP28, TP29: TP_0.75mm_SMD, kria-k26-devboard-footprints:TP_SMD_0.75mm, symbol kria-k26-devboard:TP_0.75mm_SMD
- added U31: TPS3840PL30DBVR, kria-k26-devboard-footprints:SOT-23-5, symbol kria-k26-devboard:TPS3840PH30DBVR
- C44: renamed from C60; MPN MC0402X473K160CT -> GRM155R61H474KE11D; Manufacturer Multicomp -> Murata
- C45: renamed from C61; MPN MC0402X473K160CT -> GRM155R61H474KE11D; Manufacturer Multicomp -> Murata
- TP10: renamed from TP25; now left out of the parts list
- TP11: renamed from TP26; now left out of the parts list
- TP12: renamed from TP27; now left out of the parts list
- TP9: renamed from TP24; now left out of the parts list
- renumbered C62 to C46, C63 to C47, C64 to C48, C65 to C49, C66 to C50, C67 to C51, D14 to D10, D15 to D11, R58 to R37, R59 to R38, R60 to R39, R61 to R40, R62 to R41, R63 to R42, R64 to R43, R65 to R44, R67 to R45, U17 to U14, U18 to U15, U19 to U16, U20 to U17, U21 to U18
Connections:
- net GND: now also U18.11, U18.13, U18.5, C126.2, C127.2, U31.3 (GND)
- net PS_1V8: now also R46.1, R47.1
- net PS_3V3: now also C127.1, U31.2 (VDD)
- net ~{ETH_RESET}: now also R47.2
- net ~{M2_PERST}: now also TP28.1, U31.1 (RESET); no longer R45.2, U18.2
- net ~{USB_PHY_RESET}: now also R46.2
- net CAM_RST renamed SOFTWARE_CONTROLLED_RESET
- net MIO38 renamed MIO26
- net MIO41 renamed MIO76
- net MIO44 renamed MIO77
- new net: C126.1, U31.5 (CT)
- new net ~{M2_PERST_PRE_DELAY}: R45.2, TP29.1, U18.2, U31.4 (MR_N)
- no-connect marks 6 -> 5
Other:
- moved on the sheet: R45, U18C, U18E, U18F
