File: schematics/usbc-socket.kicad_sch (KiCad schematic)
At the start: 52 parts, among them IC2 HD3SS3220RNHT, J1 Screw_Terminal_01x02, J6 USB_C_Receptacle, U23 82400152, U24 LTC4358CDE, U25 USB3310C-CP, U26 USB3310C-CP, U39 LTC4358CDE, Y3 Oscillator_24MHz_ESC_2016MV, Y7 Oscillator_24MHz_ESC_2016MV

Commit message: Voltage converter added
Parts:
- removed C110, C162: C_100n_50V_0402, kria-k26-devboard-footprints:C_0402_1005Metric, symbol kria-k26-devboard:C_100n_50V_0402
- removed C111, C112, C113, C114, C115, C116, C117, C118, C120, C121, C122, C123, C163, C164, C165: C_100n_0402, kria-k26-devboard-footprints:C_0402_1005Metric, symbol kria-k26-devboard:C_100n_0402
- removed C119, C124: C_4u7_0402, kria-k26-devboard-footprints:C_0402_1005Metric, symbol kria-k26-devboard:C_4u7_0402
- removed D16, D20: SMF4L15CA, kria-k26-devboard-footprints:SOD-123FL, symbol kria-k26-devboard:SMF4L15CA
- removed D21, D22: 1N4148WS, kria-k26-devboard-footprints:D_SOD-323F, symbol kria-k26-devboard:1N4148WS
- removed IC2: HD3SS3220RNHT, lachs_lib_kicad:QFN40P250X450X80-31N-D, symbol lachs_lib_kicad:HD3SS3220RNHT
- removed J1: Screw_Terminal_01x02, TerminalBlock_CUI:TerminalBlock_CUI_TB007-508-02_1x02_P5.08mm_Horizontal, symbol Connector:Screw_Terminal_01x02
- removed J6: USB_C_Receptacle, Connector_USB:USB_C_Receptacle_JAE_DX07S024WJ1R350, symbol Connector:USB_C_Receptacle
- removed R126: R_100R_0402, kria-k26-devboard-footprints:R_0402_1005Metric, symbol kria-k26-devboard:R_100R_0402
- removed R87, R88, R89, R90, R91, R92: R_100k_0402, kria-k26-devboard-footprints:R_0402_1005Metric, symbol kria-k26-devboard:R_100k_0402
- removed R93, R97: R_8k06_0402, kria-k26-devboard-footprints:R_0402_1005Metric, symbol kria-k26-devboard:R_8k06_0402
- removed R94, R98: R_10k_0402, kria-k26-devboard-footprints:R_0402_1005Metric, symbol kria-k26-devboard:R_10k_0402
- removed TP36, TP37, TP38, TP39, TP40, TP41, TP51, TP52: TP_0.75mm_SMD, kria-k26-devboard-footprints:TP_SMD_0.75mm, symbol kria-k26-devboard:TP_0.75mm_SMD
- removed U23: 82400152, kria-k26-devboard-footprints:SOT-563, symbol kria-k26-devboard:82400152
- removed U24, U39: LTC4358CDE, kria-k26-devboard-footprints:DFN-14-1EP_4x3mm_P0.5mm, symbol kria-k26-devboard:LTC4358CDE
- added C152, C154, C166, C167, C168, C169, C170, C171, C173, C174, C175: 100n, symbol Device:C_Small
- added C153, C172: 4u7, symbol Device:C_Small
- added J1: USB_A, symbol Connector:USB_A
- added J2: USB3_B_Micro, symbol Connector:USB3_B_Micro
- added R114, R115, R116, R117: 10k, symbol Device:R_Small
- renumbered U26 to U1, U25 to U2, Y7 to Y1, Y3 to Y2
Connections:
- net GND: now also C152.2, C153.2, C154.2, C166.2, C167.2, C168.2, C169.2, C170.2, C171.2, C172.2, C175.2, J1.4 (GND), J2.5 (GND), J2.8 (DRAIN), R115.2, R116.2; no longer U2.1 (ID)
- net GTR_DP1_C2M_N: now also J2.9 (SSRX-)
- net GTR_DP1_C2M_P: now also J2.10 (SSRX+)
- net GTR_DP1_M2C_N: now also C173.2
- net GTR_DP1_M2C_P: now also C174.2
- net GTR_DP2_M2C_C_N: now also C173.1, J2.6 (SSTX-)
- net GTR_DP2_M2C_C_P: now also C174.1, J2.7 (SSTX+)
- net MIO66: now also U1.13 (DATA2); no longer U1.18 (NXT)
- net MIO67: now also U1.18 (NXT); no longer U1.20 (STP)
- net MIO70: now also U1.20 (STP); no longer U1.13 (DATA2)
- net PS_1V8: now also C152.1, C154.1, C166.1, C168.1, C169.1, C171.1
- net SOM_5V0: now also C167.1, C170.1, J1.1 (VBUS), R117.2
- net USB2_PHY_N: now also J1.2 (D-)
- net USB2_PHY_P: now also J1.3 (D+)
- net USBC_DM: now also J2.2 (D-)
- net USBC_DP: now also J2.3 (D+)
- net at U2.2 (VBUS): now also R114.1
- net at U2.24 (RBIAS): now also R115.1
- net at U2.4 (VDD_3V3): now also C153.1
- net at U1.2 (VBUS): now also R117.1
- net at U1.24 (RBIAS): now also R116.1
- net at U1.4 (VDD_3V3): now also C172.1
- new net SHIELD: J1.SH (Shield), J2.SH (SHIELD)
- new net USB_VBUS: C175.1, J2.1 (VBUS), R114.2
- no-connect marks 9 -> 4
Other:
- note added: "USB Connector #1 - For data transfer"
- note added: "USB Connector #2 - For peripherals"
- note added: "USB-2.0 PHY #1 To handle D+/D- pins from USB-data connector"
- note added: "USB-2.0 PHY #2 For peripherals - e.g. keyboard"
- note removed: "6-15V"
- note removed: "DC JACK reverse polarity protection"
- note removed: "Power-OR Circuit"
- note removed: "USB SuperSpeed PHY"
- note removed: "USB-A 2.0 PHY"
- note removed: "USB-C 2.0 PHY"
- note removed: "USB-C connector"
- moved on the sheet: U1, U2, Y1, Y2
