File: schematics/voltage_converters.kicad_sch (KiCad schematic)
At the start: 106 parts, among them Q12 DTC014T_SOT-416, Q13 DTC014T_SOT-416, Q14 DTC014T_SOT-416, Q15 DTC014T_SOT-416, U40 RT6236AHGQUF, U41 AP62301_TSOT, U42 AP62301_TSOT, U43 AP62301_TSOT, U44 AP62301_TSOT, U45 AP62301_TSOT, U46 AP62301_TSOT, U47 AP62301_TSOT

Commit message: Voltage converter added
Parts:
- removed C166, C167: C_10u_25V_0603, kria-k26-devboard-footprints:C_0603_1608Metric, symbol kria-k26-devboard:C_10u_25V_0603
- removed C168: C_1u_0402, kria-k26-devboard-footprints:C_0402_1005Metric, symbol kria-k26-devboard:C_1u_0402
- removed C169: C_3n9_0402, kria-k26-devboard-footprints:C_0402_1005Metric, symbol kria-k26-devboard:C_3n9_0402
- removed C170, C180, C181, C182, C183, C184: C_100n_0402, kria-k26-devboard-footprints:C_0402_1005Metric, symbol kria-k26-devboard:C_100n_0402
- removed C171: C_22p_0402, kria-k26-devboard-footprints:C_0402_1005Metric, symbol kria-k26-devboard:C_22p_0402
- removed C172, C173, C174: C_22u_16V_0603, kria-k26-devboard-footprints:C_0603_1608Metric, symbol kria-k26-devboard:C_22u_16V_0603
- removed C185, C186, C187, C188, C189, C190, C191, C192: C_22u_0603, kria-k26-devboard-footprints:C_0603_1608Metric, symbol kria-k26-devboard:C_22u_0603
- removed L15: L_1u_2.6A_0806, kria-k26-devboard-footprints:L_0806_2016Metric, symbol kria-k26-devboard:L_1u_2.6A_0806
- removed L9: L_3u3_5.9A_XEL4030, kria-k26-devboard-footprints:L_Coilcraft-XEL4030, symbol kria-k26-devboard:L_3u3_6.6A_XEL4030
- removed R127: R_100k_0402, kria-k26-devboard-footprints:R_0402_1005Metric, symbol kria-k26-devboard:R_100k_0402
- removed R128, R131: R_0R_0402, kria-k26-devboard-footprints:R_0402_1005Metric, symbol kria-k26-devboard:R_0R_0402
- removed R135: R_147k_0402, kria-k26-devboard-footprints:R_0402_1005Metric, symbol kria-k26-devboard:R_147k_0402
- removed R136: R_24k_0402, kria-k26-devboard-footprints:R_0402_1005Metric, symbol kria-k26-devboard:R_24k_0402
- removed R137: R_0R_22.4A_0603, kria-k26-devboard-footprints:R_0603_1608Metric, symbol kria-k26-devboard:R_0R_22.4A_0603
- removed TP53: TP_0.75mm_SMD, kria-k26-devboard-footprints:TP_SMD_0.75mm, symbol kria-k26-devboard:TP_0.75mm_SMD
- removed U40: RT6236AHGQUF, kria-k26-devboard-footprints:UQFN-13_2x3mm_P0.5mm, symbol kria-k26-devboard:RT6236AHGQUF
- added C176, C180, C181, C182, C183: 100n, symbol Device:C_Small
- added C177, C178, C179, C184, C185, C186, C187, C188, C189: 22u, symbol Device:C_Small
- added L6: L_2u2_6.1A_XEL4030, kria-k26-devboard-footprints:L_Coilcraft-XEL4030, symbol kria-k26-devboard:L_2u2_7.8A_Coilcraft-XEL4030
- C17: renamed from C175; Val 10u/25V -> 10u; Voltage (none) -> 25V
- C18: renamed from C176; Val 10u/25V -> 10u; Voltage (none) -> 25V
- C19: renamed from C177; Val 10u/25V -> 10u; Voltage (none) -> 25V
- C20: renamed from C178; Val 10u/25V -> 10u; Voltage (none) -> 25V
- C21: renamed from C179; Val 10u/25V -> 10u; Voltage (none) -> 25V
- C35: renamed from C193; Val 10u/25V -> 10u; Voltage (none) -> 25V
- C36: renamed from C194; Val 10u/25V -> 10u; Voltage (none) -> 25V
- L1: renamed from L10; IMax (none) -> 7.8 A; ISat (none) -> 6.1 A; Val 2u2/6.1A -> 2u2/7.8A
- L2: renamed from L11; IMax (none) -> 2.6 A; ISat (none) -> 3.2 A
- L3: renamed from L12; IMax (none) -> 2.6 A; ISat (none) -> 2.9 A
- L4: renamed from L13; IMax (none) -> 2.6 A; ISat (none) -> 2.9 A
- L5: renamed from L14; IMax (none) -> 2.6 A; ISat (none) -> 3.2 A
- L7: renamed from L16; IMax (none) -> 2.6 A; ISat (none) -> 2.9 A
- R22: renamed from R151; Tolerance (none) -> template_tolerance
- R23: renamed from R152; Tolerance (none) -> template_tolerance
- R24: renamed from R153; Tolerance (none) -> template_tolerance
- R25: renamed from R154; Tolerance (none) -> template_tolerance
- R26: renamed from R155; Tolerance (none) -> template_tolerance
- R34: renamed from R161; Tolerance (none) -> template_tolerance
- R35: renamed from R162; Tolerance (none) -> template_tolerance
- TP2: renamed from TP54; now left out of the parts list
- TP3: renamed from TP55; now left out of the parts list
- TP4: renamed from TP56; now left out of the parts list
- TP5: renamed from TP57; now left out of the parts list
- TP6: renamed from TP58; now left out of the parts list
- TP7: renamed from TP59; now left out of the parts list
- TP8: renamed from TP60; now left out of the parts list
- renumbered C195 to C37, C196 to C38, C197 to C39, C198 to C40, C199 to C41, C200 to C42, D23 to D2, D25 to D3, D26 to D4, D27 to D5, D28 to D6, D29 to D7, D30 to D8, D31 to D9, Q12 to Q1, Q13 to Q2, Q14 to Q3, Q15 to Q4, R134 to R10, R141 to R11, R142 to R12, R143 to R13, R144 to R14, R145 to R15, R146 to R16, R147 to R17, R148 to R18, R149 to R19, R150 to R20, R138 to R21, R139 to R27, R140 to R28, R156 to R29, R157 to R30, R158 to R31, R159 to R32, R160 to R33, R129 to R7, R130 to R8, R132 to R9, U46 to U10, U47 to U11, U41 to U5, U42 to U6, U43 to U7, U44 to U8, U45 to U9
Connections:
- net SOM_5V_OUT is gone; now on net SOM_5V0: R9.2
- net GND: now also C177.2, C178.2, C179.2, C184.2, C185.2, C186.2, C187.2, C188.2, C189.2
- net PL_3V3_OUT: now also L6.2
- net PS_1V0_OUT: now also C189.1
- net PS_1V2_OUT: now also C187.1, C188.1
- net PS_1V8_OUT: now also C185.1, C186.1
- net PS_2V5_OUT: now also C179.1, C184.1
- net PS_3V3_OUT: now also C177.1, C178.1
- net SW_PL_3V3: now also L6.1
- net SW_PS_1V0: now also C183.2
- net SW_PS_1V2: now also C182.2
- net SW_PS_1V8: now also C181.2
- net SW_PS_2V5: now also C180.2
- net SW_PS_3V3: now also C176.2
- net at U8.6 (BST): now also C182.1
- net at U6.6 (BST): now also C180.1
- net at U7.6 (BST): now also C181.1
- net at U9.6 (BST): now also C183.1
- net at U5.6 (BST): now also C176.1
- no-connect marks 1 -> 0
Other:
- note removed: "Local FB"
- note removed: "Remote FB"
- note removed: "SOM 5V"
- moved on the sheet: C17, C18, C19, C20, C21, C35, C36, C37, C38, C39, C40, C41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
